File: pcb/dht22-atmega328.kicad_pcb (KiCad board)
At the start: 2 copper layers, 39.4 x 34.5 mm, 18 parts, among them IC1 ATMEGA328P-P, P1 CONN_01X01, P2 CONN_01X01, P3 CONN_01X01, P4 USB_B, P5 CONN_01X02, P6 CONN_01X01, P7 CONN_01X01, P8 CONN_01X01, P9 CONN_01X01, Y1 Crystal

Commit message: fix pcb
Routing:
- net Net-(IC1-Pad1): track 0.00 -> 3.15 mm
Changed lines of the file:
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@@
   (general
     (links 26)
-    (no_connects 2)
+    (no_connects 1)
     (area 139.197 89.426999 182.673584 135.615)
     (thickness 1.6)
     (drawings 8)
-    (tracks 60)
+    (tracks 62)
     (zones 0)
     (modules 18)
@@
   (segment (start 170.08094 120.904) (end 168.402 119.22506) (width 0.25) (layer B.Cu) (net 3))
   (segment (start 168.402 119.22506) (end 168.402 117.094) (width 0.25) (layer B.Cu) (net 3))
+  (segment (start 145.542 117.094) (end 145.542 119.888) (width 0.25) (layer B.Cu) (net 4) (status C00000))
+  (segment (start 145.542 119.888) (end 145.796 120.142) (width 0.25) (layer B.Cu) (net 4) (status C00000))
   (segment (start 153.162 117.094) (end 153.162 119.888) (width 0.25) (layer B.Cu) (net 7))
   (segment (start 153.162 119.888) (end 152.654 120.396) (width 0.25) (layer B.Cu) (net 7))
